Commit message: fix(swerve-sim): bind hardware arg to a property before comparing
Same xacro evaluation fix as gamora.

File: ros2/swerve_description/urdf/swerve.ros2_control.xacro (robot description, xacro)
@@ -12,11 +12,12 @@
 <robot xmlns:xacro="http://www.ros.org/wiki/xacro">
   <xacro:arg name="hardware" default="gazebo"/>
+  <xacro:property name="hardware_type" value="$(arg hardware)"/>
   <ros2_control name="SwerveSystem" type="system">
-    <xacro:if value="${$(arg hardware) == 'mock'}">
+    <xacro:if value="${hardware_type == 'mock'}">
       <hardware>
         <plugin>mock_components/GenericSystem</plugin>
       </hardware>
     </xacro:if>
-    <xacro:if value="${$(arg hardware) == 'gazebo'}">
+    <xacro:if value="${hardware_type == 'gazebo'}">
       <hardware>
         <plugin>gz_ros2_control/GazeboSimSystem</plugin>
